File: KiCad/K9AY_switch/K9AY_switch.kicad_pcb (KiCad board)
At the start: 2 copper layers, 144.1 x 108.1 mm, 137 parts, among them J3 LOOPS, J4 12V, J5 USB_B_Micro, J6 RF_OUT, J7 MANUAL_SWITCH, K1 G5V-2, K10 TIANBO-HJR-4102-L, K11 TIANBO-HJR-4102-L, K12 TIANBO-HJR-4102-L, K2 G5V-2, K3 G5V-2, K4 G5V-2, K5 TIANBO-HJR-4102-L, K6 TIANBO-HJR-4102-L, K7 TIANBO-HJR-4102-L, K8 TIANBO-HJR-4102-L, K9 TIANBO-HJR-4102-L, Q1 MMBFJ310, Q2 BC817, Q3 BC817, Q4 MMBFJ310, Q5 IRLML5203, U1 ESP-12F, U11 CH340C, U12 USBLC6, U2 74HC595, U3 74HC595, U4 ULN2003A, U5 L7803, U6 L7805, U7 74HC04, U8 ULN2003A

Commit message: Update KiCad project, gerbers and pictures
- updated schematic, PCB, BOM, gerbers and plots
- new photos: k1, mosfet, pwr; updated direction diagram
- ignore KiCad backups, *.tar.gz and k9ay_v5.zip

Co-Authored-By: Claude Opus 5.5 <noreply@anthropic.com>
Parts:
- added C30: 47uF, Capacitor_THT:CP_Radial_D5.0mm_P2.50mm, F.Cu at (180.1, 102.1)
- added C32: 10u, Capacitor_SMD:C_1206_3216Metric, F.Cu at (187.5, 103.1)
- added C35: 100n, Capacitor_SMD:C_1206_3216Metric, F.Cu at (182.4, 117.3)
- added C36: 100n, Capacitor_SMD:C_1206_3216Metric, F.Cu at (182.4, 120.1)
- added L2: 470uH, Inductor_THT:L_Radial_D10.0mm_P5.00mm_Neosid_SD12_style3, F.Cu at (189.7, 66.8)
- added L3: 470uH, Inductor_THT:L_Radial_D10.0mm_P5.00mm_Neosid_SD12_style3, F.Cu at (185.0, 77.7)
- added L4: 470uH, Inductor_THT:L_Radial_D10.0mm_P5.00mm_Neosid_SD12_style3, F.Cu at (167.2, 117.1)
- K3: value G5V-2 -> Tianbo HJR 1-2C-12V
- U5: value L7803 -> K7803-500R3
- U6: value L7805 -> K7805-500R3
- moved C8 4.23 mm to (175.9, 109.0)
- moved C9 3.92 mm to (171.9, 109.0)
- moved R1 2.86 mm to (165.6, 124.4)
- moved D2 2.86 mm to (170.7, 124.5)
- moved C29 2.10 mm to (169.1, 109.1)
- moved C27 2.10 mm to (163.9, 109.1)
- moved C28 2.10 mm to (166.5, 109.1)
- moved C7 2.10 mm to (180.1, 110.5)
- moved C2 1.24 mm to (173.7, 82.5)
Connections:
- C10 pad 1: 5V -> Net-(U6-VO)
- C11 pad 1: 5V -> Net-(U6-VO)
- C22 pad 1: 12V -> Net-(U6-VI)
- C23 pad 1: 12V -> Net-(U6-VI)
- U6 pad 1: 12V -> Net-(U6-VI)
- U6 pad 3: 5V -> Net-(U6-VO)
Routing:
- net Net-(U6-VI): track 0.00 -> 91.6 mm
- net Net-(C30-Pad1): track 0.00 -> 45.8 mm
- net Net-(U6-VO): track 0.00 -> 23.0 mm
- net 12V: track 474.1 -> 459.0 mm
- net GND: track 575.0 -> 588.7 mm, vias 21 -> 23
- net 3.3V: track 183.2 -> 186.3 mm
- net 5V: track 451.6 -> 449.1 mm, vias 12 -> 14
Other:
- board text removed: "PWR"
